File: Gerber/quadcopter.brd (EAGLE design)
At the start: 137.2 x 137.2 mm, 67 parts, among them J4 AVR_SPI_PRG_6NS, U2 ATMEGA128RFA1

Commit message: Finish
Routing:
- net TX0: track 62.1 -> 64.6 mm
- net SDA: track 71.5 -> 73.7 mm
- net RX0: track 75.6 -> 77.6 mm
- net VBAT: track 141.1 -> 143.0 mm
- net PE4: track 126.8 -> 128.5 mm
- net SCL: track 90.5 -> 92.1 mm
- net GND: track 359.2 -> 360.2 mm
- net PE3: track 100.0 -> 100.9 mm
- net RESET: track 124.8 -> 124.3 mm
