File: designRules/quadcopter.brd (EAGLE design)
At the start: 137.2 x 137.2 mm, 67 parts, among them J4 AVR_SPI_PRG_6NS, SW1 PUSHBUTTON_SMD-VERTICAL-1, U2 ATMEGA128RFA1

Commit message: Board finally passes DFM
Parts:
- moved SW1 127.9 mm to (-86.3, -74.5), turned to 0 degrees
- moved C14 2.29 mm to (-17.5, -20.0)
- moved C16 1.91 mm to (-16.4, -13.4)
- moved C18 1.91 mm to (-12.8, -13.4)
- moved Y2 1.91 mm to (-14.4, -16.7)
- moved R3 1.21 mm to (-6.10, -1.65)
- moved C28 0.95 mm to (-5.27, 6.35)
- moved R2 0.70 mm to (-6.35, 0.32)
- moved C31 0.70 mm to (-0.13, 6.35)
Connections:
- new net N$3: SW1.1, SW1.2
- new net N$6: SW1.3, SW1.4
- net BAT_GND: now also U$1.P$2, U$2.P$2, U$3.P$2, U$4.P$2; no longer U$1.P$5, U$2.P$5, U$3.P$5, U$4.P$5
- net FILTERED1: now also U$4.P$1; no longer U$4.P$4
- net FILTERED2: now also U$2.P$1; no longer U$2.P$4
- net FILTERED3: now also U$3.P$1; no longer U$3.P$4
- net FILTERED4: now also U$1.P$1; no longer U$1.P$4
- net FLYBACK1: now also U$4.P$3; no longer U$4.P$1
- net FLYBACK2: now also U$2.P$3; no longer U$2.P$1
- net FLYBACK3: now also U$3.P$3; no longer U$3.P$1
- net FLYBACK4: now also U$1.P$3; no longer U$1.P$1
- net GND: no longer SW1.3, SW1.4
- net RESET: no longer SW1.1, SW1.2
Routing:
- net GND: track 341.1 -> 403.0 mm, vias 19 -> 23
- net 3.0V: track 260.9 -> 232.2 mm, vias 3 -> 7
- net PE3: track 107.7 -> 81.3 mm
- net SCL: track 76.7 -> 99.9 mm, vias 2 -> 4
- net RESET: track 142.4 -> 119.8 mm, vias 1 -> 2
- net BAT_GND: track 81.9 -> 101.7 mm, vias 4 -> 8
- net PB5: track 92.6 -> 78.8 mm, vias 0 -> 2
- net VBAT: track 126.8 -> 139.5 mm, vias 6 -> 11
- net TX0: track 91.2 -> 78.8 mm
- net MOSI: track 50.2 -> 62.0 mm, vias 0 -> 1
- net N$6: track 0.00 -> 9.20 mm
- net N$3: track 0.00 -> 9.14 mm
- net SDA: track 79.2 -> 70.7 mm
- net PE5: track 93.8 -> 101.3 mm, vias 2 -> 1
- net RX0: track 74.4 -> 80.8 mm
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- added copper zone on layer 1, net N$8
- removed copper zone on layer 1, net GND
